File: hardwarebs/MobileArkhamAsylum.kicad_pcb (KiCad board)
At the start: 2 copper layers, 142.5 x 72.5 mm, 25 parts, among them J1 Conn_01x03_Pin, J2 Conn_01x02_Socket, J3 Conn_01x08_Pin, J4 Conn_01x02_Pin, J5 Conn_Receptacle_2P, Q1 NMOS, U1 R-78C3.3-1.0, U2 BQ24079RGT, U3 R-78C5.0-1.0

Commit message: v2 footprint and design
Parts:
- C2, C3, C4, C5: footprint Capacitor_THT:CP_Radial_D5.0mm_P2.00mm -> Capacitor_THT:CP_Radial_D5.0mm_P2.50mm
- Q1: footprint Transistor_Power:GaN_Systems_GaNPX-3_5x6.6mm_Drain3.76x0.6mm -> Package_TO_SOT_SMD:SOT-23
Routing:
- net Net-(J5-L): track 48.0 -> 29.1 mm, vias 4 -> 2
- net /NMOS G: track 66.8 -> 68.0 mm
- net GND: track 298.4 -> 297.8 mm
