File: hardwarebs/MobileArkhamAsylum.kicad_sch (KiCad schematic)
At the start: 25 parts, among them J1 Conn_01x03_Pin, J2 Conn_01x02_Socket, J3 Conn_01x08_Pin, J4 Conn_01x02_Pin, J5 Conn_Receptacle_2P, Q1 NMOS, U1 R-78C3.3-1.0, U2 BQ24079RGT, U3 R-78C5.0-1.0

Commit message: v2 footprint and design
Parts:
- C2, C3, C4, C5: footprint Capacitor_THT:CP_Radial_D5.0mm_P2.00mm -> Capacitor_THT:CP_Radial_D5.0mm_P2.50mm
- Q1: footprint Transistor_Power:GaN_Systems_GaNPX-3_5x6.6mm_Drain3.76x0.6mm -> Package_TO_SOT_SMD:SOT-23
Changed lines of the file:
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@@
 			)
 		)
-		(property "Footprint" "Transistor_Power:GaN_Systems_GaNPX-3_5x6.6mm_Drain3.76x0.6mm"
+		(property "Footprint" "Package_TO_SOT_SMD:SOT-23"
 			(at 142.24 115.57 0)
 			(effects
@@
 			)
 		)
-		(property "Footprint" "Capacitor_THT:CP_Radial_D5.0mm_P2.00mm"
+		(property "Footprint" "Capacitor_THT:CP_Radial_D5.0mm_P2.50mm"
 			(at 125.4252 76.2 0)
 			(effects
@@
 			)
 		)
-		(property "Footprint" "Capacitor_THT:CP_Radial_D5.0mm_P2.00mm"
+		(property "Footprint" "Capacitor_THT:CP_Radial_D5.0mm_P2.50mm"
 			(at 156.21 56.8452 0)
 			(effects
@@
 			)
 		)
-		(property "Footprint" "Capacitor_THT:CP_Radial_D5.0mm_P2.00mm"
+		(property "Footprint" "Capacitor_THT:CP_Radial_D5.0mm_P2.50mm"
 			(at 114.3 56.8452 0)
 			(effects
@@
 			)
 		)
-		(property "Footprint" "Capacitor_THT:CP_Radial_D5.0mm_P2.00mm"
+		(property "Footprint" "Capacitor_THT:CP_Radial_D5.0mm_P2.50mm"
 			(at 154.94 76.5048 0)
 			(effects
